File: Boarddevelop/Mainv1/Mainv1.kicad_sch (KiCad schematic)
At the start: 0 parts

Commit message: PCB update
updated ACD
Other:
- added sheet ACD (ACD.kicad_sch)
Changed lines of the file:
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@@
 	(generator_version "9.0")
 	(paper "A4")
+	(sheet
+		(at 17.78 17.78)
+		(size 12.7 5.08)
+		(exclude_from_sim no)
+		(in_bom yes)
+		(on_board yes)
+		(dnp no)
+		(fields_autoplaced yes)
+		(stroke
+			(width 0.1)
+			(type solid)
+		)
+		(fill
+			(color 0 0 0 0.0000)
+		)
+		(property "Sheetname" "ACD"
+			(at 17.78 -482.8554 0)
+			(show_name yes)
+			(effects
+				(font
+					(size 1.27 1.27)
+				)
+				(justify left bottom)
+			)
+		)
+		(property "Sheetfile" "ACD.kicad_sch"
+			(at 17.78 523.3684 0)
+			(show_name yes)
+			(effects
+				(font
+					(size 1.27 1.27)
+				)
+				(justify left top)
+			)
+		)
+		(instances
+			(project "Mainv1"
+				(path "/2f9812ee-cc02-4b04-baa3-83e13ffe25be"
+					(page "2")
+				)
+			)
+		)
+	)
 	(sheet_instances
 		(path "/"
